File: test.kicad_pcb (KiCad board)
At the start: 2 copper layers, 12 parts, among them J1 Conn_01x03_Male, U1 slider-20

Commit message: update 0625
とりま基板完成？
Parts:
- removed J1: Conn_01x03_Male, Pin_Headers:Pin_Header_Angled_1x03_Pitch2.54mm
- added C1: 0.1u, Capacitor_SMD:C_0603_1608Metric_Pad0.99x1.00mm_HandSolder, B.Cu at (118.0, 61.6)
- added C10: 22u, Capacitor_SMD:C_0805_2012Metric_Pad1.29x1.40mm_HandSolder, B.Cu at (162.4, 81.3)
- added C11: 22u, Capacitor_SMD:C_0805_2012Metric_Pad1.29x1.40mm_HandSolder, B.Cu at (131.4, 80.4)
- added C12: 22u, Capacitor_SMD:C_0805_2012Metric_Pad1.29x1.40mm_HandSolder, B.Cu at (192.2, 81.9)
- added C13: 22u, Capacitor_SMD:C_0805_2012Metric_Pad1.29x1.40mm_HandSolder, B.Cu at (133.9, 80.4)
- added C14: 22u, Capacitor_SMD:C_0805_2012Metric_Pad1.29x1.40mm_HandSolder, B.Cu at (112.3, 71.9)
- added C15: 0.1u, Capacitor_SMD:C_0805_2012Metric_Pad1.29x1.40mm_HandSolder, B.Cu at (132.3, 77.2)
- added C16: 0.1u, Capacitor_SMD:C_0805_2012Metric_Pad1.29x1.40mm_HandSolder, B.Cu at (129.2, 73.7)
- added C17: 47u, Capacitor_SMD:CP_Elec_6.3x4.5, B.Cu at (127.6, 61.5)
- added C2: 0.1u, Capacitor_SMD:C_0603_1608Metric_Pad0.99x1.00mm_HandSolder, B.Cu at (160.2, 79.6)
- added C3: 0.1u, Capacitor_SMD:C_0603_1608Metric_Pad0.99x1.00mm_HandSolder, B.Cu at (136.6, 81.1)
- added C4: 0.1u, Capacitor_SMD:C_0603_1608Metric_Pad0.99x1.00mm_HandSolder, B.Cu at (184.0, 79.3)
- added C5: 22u, Capacitor_SMD:C_0805_2012Metric_Pad1.29x1.40mm_HandSolder, B.Cu at (159.6, 82.4)
- added C6: 22u, Capacitor_SMD:C_0805_2012Metric_Pad1.29x1.40mm_HandSolder, B.Cu at (189.5, 82.0)
- added C7: 22u, Capacitor_SMD:C_0805_2012Metric_Pad1.29x1.40mm_HandSolder, B.Cu at (183.2, 81.9)
- added C8: 22u, Capacitor_SMD:C_0805_2012Metric_Pad1.29x1.40mm_HandSolder, B.Cu at (186.8, 82.0)
- added C9: 22u, Capacitor_SMD:C_0805_2012Metric_Pad1.29x1.40mm_HandSolder, B.Cu at (136.5, 78.3)
- added D1: LED, mTouch:LED_0603_1608Metric_Pad_ReverseMounted, B.Cu at (116.5, 41.9)
- added D10: LED, mTouch:LED_0603_1608Metric_Pad_ReverseMounted, B.Cu at (152.5, 41.9)
- added D11: LED, mTouch:LED_0603_1608Metric_Pad_ReverseMounted, B.Cu at (149.0, 42.0)
- added D12: LED, mTouch:LED_0603_1608Metric_Pad_ReverseMounted, B.Cu at (156.0, 41.9)
- added D13: LED, mTouch:LED_0603_1608Metric_Pad_ReverseMounted, B.Cu at (159.5, 41.9)
- added D14: LED, mTouch:LED_0603_1608Metric_Pad_ReverseMounted, B.Cu at (163.0, 41.9)
- added D15: LED, mTouch:LED_0603_1608Metric_Pad_ReverseMounted, B.Cu at (166.5, 41.9)
- added D16: LED, mTouch:LED_0603_1608Metric_Pad_ReverseMounted, B.Cu at (170.0, 41.9)
- added D17: LED, mTouch:LED_0603_1608Metric_Pad_ReverseMounted, B.Cu at (173.5, 41.9)
- added D18: LED, mTouch:LED_0603_1608Metric_Pad_ReverseMounted, B.Cu at (177.0, 41.9)
- added D19: LED, mTouch:LED_0603_1608Metric_Pad_ReverseMounted, B.Cu at (187.5, 41.9)
- added D2: LED, mTouch:LED_0603_1608Metric_Pad_ReverseMounted, B.Cu at (131.5, 41.9)
- added D20: LED, mTouch:LED_0603_1608Metric_Pad_ReverseMounted, B.Cu at (197.6, 41.9)
- added D3: LED, mTouch:LED_0603_1608Metric_Pad_ReverseMounted, B.Cu at (123.5, 41.9)
- added D4: LED, mTouch:LED_0603_1608Metric_Pad_ReverseMounted, B.Cu at (138.5, 41.9)
- added D5: LED, mTouch:LED_0603_1608Metric_Pad_ReverseMounted, B.Cu at (119.9, 41.9)
- added D6: LED, mTouch:LED_0603_1608Metric_Pad_ReverseMounted, B.Cu at (135.0, 41.9)
- added D7: LED, mTouch:LED_0603_1608Metric_Pad_ReverseMounted, B.Cu at (127.5, 41.9)
- added D8: LED, mTouch:LED_0603_1608Metric_Pad_ReverseMounted, B.Cu at (142.0, 41.9)
- added D9: LED, mTouch:LED_0603_1608Metric_Pad_ReverseMounted, B.Cu at (145.5, 41.9)
- added JP1: Regulator, Jumper:SolderJumper-2_P1.3mm_Open_RoundedPad1.0x1.5mm, B.Cu at (126.7, 73.8)
- added L1: 10uH, Inductor_SMD:L_6.3x6.3_H3, B.Cu at (128.2, 68.8)
- added Q1: SKI03036, Package_TO_SOT_SMD:TO-263-2, B.Cu at (150.2, 76.7)
- added Q2: SKI03036, Package_TO_SOT_SMD:TO-263-2, B.Cu at (173.7, 76.2)
- added Q3: SKI03036, Package_TO_SOT_SMD:TO-263-2, B.Cu at (198.0, 76.3)
- added R11: 10, Resistor_SMD:R_0603_1608Metric_Pad0.99x1.00mm_HandSolder, B.Cu at (187.3, 79.3)
- added REF**: t, mTouch:TestPoint_Pad_D1.5mm, B.Cu at (111.8, 80.0)
- added REF**: MountingHole_3.2mm_M3_DIN965, MountingHole:MountingHole_3.2mm_M3_DIN965, F.Cu at (110.7, 40.2)
- added REF**: MountingHole_3.2mm_M3_DIN965, MountingHole:MountingHole_3.2mm_M3_DIN965, F.Cu at (205.4, 84.8)
- added REF**: t, mTouch:TestPoint_Pad_D1.5mm, B.Cu at (114.3, 82.5)
- added REF**: t, mTouch:TestPoint_Pad_D1.5mm, B.Cu at (116.8, 82.5)
- added REF**: t, mTouch:TestPoint_Pad_D1.5mm, B.Cu at (116.8, 80.0)
- added REF**: t, mTouch:TestPoint_Pad_D1.5mm, B.Cu at (114.3, 80.0)
- added REF**: t, mTouch:TestPoint_Pad_D1.5mm, B.Cu at (116.8, 77.5)
- added REF**: t, mTouch:TestPoint_Pad_D1.5mm, B.Cu at (114.3, 77.5)
- added REF**: MountingHole_3.2mm_M3_DIN965, MountingHole:MountingHole_3.2mm_M3_DIN965, F.Cu at (110.7, 84.9)
- added REF**: MountingHole_3.2mm_M3_DIN965, MountingHole:MountingHole_3.2mm_M3_DIN965, F.Cu at (205.5, 40.1)
- added TP1: ~MCLR, mTouch:TestPoint_Pad_D1.5mm, B.Cu at (109.7, 77.3)
- added TP2: Vcc, mTouch:TestPoint_Pad_D1.5mm, B.Cu at (111.8, 74.9)
- added TP2: 5V, mTouch:TestPoint_Pad_D1.5mm, B.Cu at (115.3, 72.9)
- added TP2: Vcc, mTouch:TestPoint_Pad_D1.5mm, B.Cu at (109.7, 74.9)
- added TP3: GND, mTouch:TestPoint_Pad_D1.5mm, B.Cu at (111.8, 77.5)
- added TP3: GND, mTouch:TestPoint_Pad_D1.5mm, B.Cu at (116.8, 85.1)
- added TP3: GND, mTouch:TestPoint_Pad_D1.5mm, B.Cu at (109.7, 72.4)
- added TP4: DAT, mTouch:TestPoint_Pad_D1.5mm, B.Cu at (109.7, 67.3)
- added TP5: CLK, mTouch:TestPoint_Pad_D1.5mm, B.Cu at (109.7, 69.8)
- added TP6: CdS, TestPoint:TestPoint_Pad_D1.5mm, B.Cu at (116.8, 74.9)
- added TP7: DebugTx, TestPoint:TestPoint_Pad_D1.5mm, B.Cu at (114.3, 74.9)
- added U2: TLP152, Package_SO:MFSOP6-5_4.4x3.6mm_P1.27mm, B.Cu at (139.4, 75.8)
- added U3: TLP152, Package_SO:MFSOP6-5_4.4x3.6mm_P1.27mm, B.Cu at (161.5, 74.5)
- added U4: TLP152, Package_SO:MFSOP6-5_4.4x3.6mm_P1.27mm, B.Cu at (185.9, 73.8)
- added U5: touchSlider5, mTouch:mTouch3-1, F.Cu at (156.8, 51.6)
- added U6: NJU7223, Package_TO_SOT_SMD:TO-252-2, B.Cu at (124.3, 78.8)
- R1, R2, R3, R4, R5: value 33k -> 33; footprint Resistors_SMD:R_0603_HandSoldering -> Resistor_SMD:R_0603_1608Metric_Pad0.99x1.00mm_HandSolder
- R10, R9: value 33k -> 10; footprint Resistors_SMD:R_0603_HandSoldering -> Resistor_SMD:R_0603_1608Metric_Pad0.99x1.00mm_HandSolder
- R6, R7, R8: value 33k -> 220; footprint Resistors_SMD:R_0603_HandSoldering -> Resistor_SMD:R_0603_1608Metric_Pad0.99x1.00mm_HandSolder
- U1: value slider-20 -> PIC16F1933; footprint mTouch:Slider-20 -> Package_SO:SSOP-20_5.3x7.2mm_P0.65mm; moved to B.Cu
- moved R5 53.2 mm to (112.6, 64.6)
- moved R4 49.4 mm to (112.6, 63.1)
- moved R9 45.0 mm to (139.9, 81.1), turned to 180 degrees
- moved U1 43.8 mm to (119.6, 67.6), turned to 90 degrees
- moved R3 42.5 mm to (112.6, 66.1)
- moved R2 42.5 mm to (112.7, 61.5)
- moved R1 41.0 mm to (112.7, 60.0)
- moved R7 36.3 mm to (143.3, 71.7)
- moved R8 32.5 mm to (189.9, 70.7)
- moved R10 31.3 mm to (163.5, 79.7), turned to 180 degrees
- moved R6 28.4 mm to (165.7, 71.2)
Connections:
- R1 pad 1: /SE -> Net-(D1-Pad1)
- R1 pad 2: Net-(R1-Pad2) -> /ILED1
- R10 pad 1: Net-(R10-Pad1) -> Net-(Q2-Pad1)
- R10 pad 2: /SE -> Net-(R10-Pad2)
- R2 pad 1: Net-(R1-Pad2) -> Net-(D1-Pad2)
- R2 pad 2: Net-(R2-Pad2) -> /ILED2
- R3 pad 1: Net-(R2-Pad2) -> Net-(D10-Pad1)
- R3 pad 2: /S1 -> /ILED3
- R4 pad 1: /S1 -> Net-(D13-Pad2)
- R4 pad 2: Net-(R4-Pad2) -> /ILED4
- R5 pad 1: Net-(R4-Pad2) -> Net-(D10-Pad2)
- R5 pad 2: Net-(R5-Pad2) -> /ILED5
- R6 pad 1: Net-(R5-Pad2) -> Net-(R6-Pad1)
- R6 pad 2: /S2 -> GND
- R7 pad 1: /S2 -> Net-(R7-Pad1)
- R7 pad 2: Net-(R7-Pad2) -> GND
- R8 pad 1: Net-(R7-Pad2) -> Net-(R8-Pad1)
- R8 pad 2: Net-(R8-Pad2) -> GND
- R9 pad 1: Net-(R8-Pad2) -> Net-(Q1-Pad1)
- R9 pad 2: Net-(R10-Pad1) -> Net-(R9-Pad2)
- U1 pad 1: /SE -> /ILED4
- U1 pad 10: Net-(R10-Pad1) -> /ILED3
- U1 pad 2: Net-(R1-Pad2) -> /PWM3
- U1 pad 3: Net-(R2-Pad2) -> /CdS
- U1 pad 4: /S1 -> /IRsens
- U1 pad 5: Net-(R4-Pad2) -> GNDD
- U1 pad 6: Net-(R5-Pad2) -> GNDD
- U1 pad 7: /S2 -> /PWM1
- U1 pad 8: Net-(R7-Pad2) -> /ILED5
- U1 pad 9: Net-(R8-Pad2) -> /DebugTx
Routing:
- net +12V: track 0.00 -> 279.6 mm, vias 0 -> 38
- net GND: track 0.00 -> 208.5 mm, vias 0 -> 76
- net Net-(U1-Pad20): track 0.00 -> 122.7 mm, vias 0 -> 3
- net Net-(D10-Pad2): track 0.00 -> 122.4 mm, vias 0 -> 2
- net Net-(D1-Pad1): track 0.00 -> 116.6 mm, vias 0 -> 2
- net /SE: track 100.7 -> 0.00 mm, vias 2 -> 0
- net Net-(D1-Pad2): track 0.00 -> 100.7 mm, vias 0 -> 2
- net Net-(TP5-Pad1): track 0.00 -> 94.1 mm, vias 0 -> 3
- net Net-(D13-Pad2): track 0.00 -> 88.3 mm, vias 0 -> 4
- net Net-(D10-Pad1): track 0.00 -> 84.0 mm, vias 0 -> 6
- net /PWM3: track 0.00 -> 76.2 mm
- net Net-(TP4-Pad1): track 0.00 -> 74.4 mm, vias 0 -> 5
- net +5VD: track 0.00 -> 51.9 mm, vias 0 -> 8
- net Net-(U1-Pad12): track 0.00 -> 48.3 mm, vias 0 -> 3
- net /PWM2: track 0.00 -> 47.5 mm, vias 0 -> 2
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- added copper zone on B.Cu, net +12V
- added copper zone on F.Cu, net +12V
- added copper zone on B.Cu, net /O1
- added copper zone on F.Cu, net /O1
- added copper zone on B.Cu, net /O2
- added copper zone on F.Cu, net /O2
- added copper zone on B.Cu, net /O3
- added copper zone on F.Cu, net /O3
- added copper zone on B.Cu, net GND
- added copper zone on F.Cu, net GND
- added copper zone on B.Cu, net GNDD
- added copper zone on F.Cu, net GNDD
Other:
- board outline added: 99.9 x 49.8 mm
- net class DigitalPower added: clearance 0.2, trace_width 0.4, via_dia 0.9, via_drill 0.5
- net class Power added: clearance 0.2, trace_width 0.5, via_dia 1, via_drill 0.7
- net class touch added: clearance 0.2, trace_width 0.25, via_dia 0.8, via_drill 0.4
- board text added: "15V->3V3"
- board text added: "6A/ch 12A(Total)"
- board text added: "CH1"
- board text added: "CH2"
- board text added: "CH3"
- board text added: "PIC 16F1827"
- board text added: "TX"

Commit message: update
Parts:
- added C18: 100u 12.5V, Capacitors_Tantalum_SMD:CP_Tantalum_Case-X_EIA-7343-43_Hand, B.Cu at (191.8, 61.0)
- added C19: 100u 12.5V, Capacitors_Tantalum_SMD:CP_Tantalum_Case-X_EIA-7343-43_Hand, B.Cu at (179.8, 61.0)
- added MK1: Mounting_Hole_PAD, TestPoint:TestPoint_Pad_D1.0mm, F.Cu at (170.9, 101.8)
- added MK2: Mounting_Hole_PAD, TestPoint:TestPoint_Pad_D1.0mm, F.Cu at (170.9, 106.9)
- added MK3: Mounting_Hole_PAD, TestPoint:TestPoint_Pad_D1.0mm, F.Cu at (185.9, 101.8)
- added MK4: Mounting_Hole_PAD, TestPoint:TestPoint_Pad_D1.0mm, F.Cu at (170.9, 111.9)
- added MK5: Mounting_Hole_PAD, TestPoint:TestPoint_Pad_D1.0mm, F.Cu at (185.9, 106.9)
- added MK6: Mounting_Hole_PAD, TestPoint:TestPoint_Pad_D1.0mm, F.Cu at (170.9, 117.0)
- added MK7: Mounting_Hole_PAD, TestPoint:TestPoint_Pad_D1.0mm, F.Cu at (185.9, 111.9)
- added MK8: Mounting_Hole_PAD, TestPoint:TestPoint_Pad_D1.0mm, F.Cu at (185.9, 117.0)
- C10, C5: moved to F.Cu
- moved C10 42.6 mm to (199.6, 102.0)
- moved C5 40.9 mm to (195.5, 102.0), turned to 0 degrees
Routing:
- net +12V: track 279.6 -> 148.3 mm, vias 38 -> 14
- net GND: track 208.5 -> 258.4 mm, vias 76 -> 71
- net /O1: track 46.5 -> 56.7 mm, vias 9 -> 12
- net Net-(C18-Pad2): track 0.00 -> 4.39 mm
- net GNDD: track 26.8 -> 29.7 mm, vias 10 -> 11
Other:
- net class Power: trace_width 0.5 -> 1.5; via_dia 1 -> 0.8; via_drill 0.7 -> 0.4
