File: test.sch (KiCad schematic (older format))
At the start: 12 parts, among them J1 Conn_01x03_Male, U1 slider-20

Commit message: update 0625
とりま基板完成？
Parts:
- removed J1: Conn_01x03_Male, Pin_Headers:Pin_Header_Angled_1x03_Pitch2.54mm, symbol Connector:Conn_01x03_Male
- removed U1: slider-20, mTouch:Slider-20, symbol mtouch:slider-20
- added C1, C2, C3, C4: 0.1u, Capacitor_SMD:C_0603_1608Metric_Pad0.99x1.00mm_HandSolder, symbol Device:C_Small
- added C10, C11, C12, C13, C14, C5, C6, C7, C8, C9: 22u, Capacitor_SMD:C_0805_2012Metric_Pad1.29x1.40mm_HandSolder, symbol Device:C_Small
- added C15, C16: 0.1u, Capacitor_SMD:C_0805_2012Metric_Pad1.29x1.40mm_HandSolder, symbol Device:C_Small
- added C17: 47u, Capacitor_SMD:CP_Elec_6.3x4.5, symbol Device:CP_Small
- added D1, D10, D11, D12, D13, D14, D15, D16, D17, D18, D19, D2, D20, D3, D4, D5, D6, D7, D8, D9: LED, mTouch:LED_0603_1608Metric_Pad_ReverseMounted, symbol Device:LED_Small
- added JP1: Regulator, Jumper:SolderJumper-2_P1.3mm_Open_RoundedPad1.0x1.5mm, symbol Device:Jumper_NO_Small
- added L1: 10uH, Inductor_SMD:L_6.3x6.3_H3, symbol pspice:INDUCTOR
- added MK1, MK2, MK3, MK4, MK5, MK6, MK7, MK8: Mounting_Hole_PAD, TestPoint:TestPoint_Pad_D1.0mm, symbol Mechanical:Mounting_Hole_PAD
- added Q1, Q2, Q3: SKI03036, Package_TO_SOT_SMD:TO-263-2, symbol Device:Q_NMOS_GDS
- added R11: 10, Resistor_SMD:R_0603_1608Metric_Pad0.99x1.00mm_HandSolder, symbol Device:R_Small
- added TP1: ~MCLR, TestPoint:TestPoint_Pad_D1.5mm, symbol Connector:Test_Point
- added TP2: Vcc, TestPoint:TestPoint_Pad_D1.5mm, symbol Connector:Test_Point
- added TP3: GND, TestPoint:TestPoint_Pad_D1.5mm, symbol Connector:Test_Point
- added TP4: DAT, TestPoint:TestPoint_Pad_D1.5mm, symbol Connector:Test_Point
- added TP5: CLK, TestPoint:TestPoint_Pad_D1.5mm, symbol Connector:Test_Point
- added TP6: CdS, TestPoint:TestPoint_Pad_D1.5mm, symbol Connector:Test_Point
- added TP7: DebugTx, TestPoint:TestPoint_Pad_D1.5mm, symbol Connector:Test_Point
- added U1: PIC16F1933, Package_SO:SSOP-20_5.3x7.2mm_P0.65mm, symbol PIC:PIC16F1933
- added U2, U3, U4: TLP152, Package_SO:MFSOP6-5_4.4x3.6mm_P1.27mm, symbol Isolator:TLP2767
- added U5: touchSlider5, mTouch:mTouch3-1, symbol slider:touchSlider5
- added U6: NJU7223, Package_TO_SOT_SMD:TO-252-2, symbol Regulator_Linear:LM3480-3.3
- R1, R2, R3, R4, R5: value 33k -> 33; footprint Resistors_SMD:R_0603_HandSoldering -> Resistor_SMD:R_0603_1608Metric_Pad0.99x1.00mm_HandSolder
- R10, R9: value 33k -> 10; footprint Resistors_SMD:R_0603_HandSoldering -> Resistor_SMD:R_0603_1608Metric_Pad0.99x1.00mm_HandSolder
- R6, R7, R8: value 33k -> 220; footprint Resistors_SMD:R_0603_HandSoldering -> Resistor_SMD:R_0603_1608Metric_Pad0.99x1.00mm_HandSolder
Connections:
- net labels added: +12V, +5VD, CdS, DebugTx, GND, GNDD, ILED1, ILED2, ILED3, ILED4, ILED5, IRsens, O1, O2, O3, PWM1, PWM2, PWM3
- net labels removed: S1, S2, SE
- wire segments 68 -> 187

Commit message: update
Parts:
- added C18, C19: 100u 12.5V, Capacitor_SMD:CP_Elec_6.3x4.5, symbol Device:CP_Small
Connections:
- wire segments 187 -> 196
Changed lines of the file:
@@
 Connection ~ 4700 4750
 Wire Wire Line
-	5050 4750 5400 4750
+	5050 4750 5300 4750
 Connection ~ 5050 4750
 Wire Wire Line
-	5400 4950 5050 4950
+	5400 4950 5300 4950
 Connection ~ 5050 4950
 $Comp
@@
 Wire Wire Line
 	2600 2750 5150 2750
+$Comp
+L Device:CP_Small C19
+U 1 1 5B32FFC6
+P 6050 5000
+F 0 "C19" H 5962 4954 50  0000 R CNN
+F 1 "100u 12.5V" H 6500 5100 50  0000 R CNN
+F 2 "Capacitor_SMD:CP_Elec_6.3x4.5" H 6050 5000 50  0001 C CNN
+F 3 "~" H 6050 5000 50  0001 C CNN
+	1    6050 5000
+	1    0    0    -1
+$EndComp
+$Comp
+L Device:CP_Small C18
+U 1 1 5B33041D
+P 6050 4750
+F 0 "C18" H 5962 4704 50  0000 R CNN
+F 1 "100u 12.5V" H 6500 4850 50  0000 R CNN
+F 2 "Capacitor_SMD:CP_Elec_6.3x4.5" H 6050 4750 50  0001 C CNN
+F 3 "~" H 6050 4750 50  0001 C CNN
+	1    6050 4750
+	1    0    0    -1
+$EndComp
+Wire Wire Line
+	6050 4850 6050 4900
+Wire Wire Line
+	6050 4650 6050 4600
+Wire Wire Line
+	6050 4600 5300 4600
+Wire Wire Line
+	5300 4600 5300 4750
+Connection ~ 5300 4750
+Wire Wire Line
+	5300 4750 5400 4750
+Wire Wire Line
+	5300 4950 5300 5150
+Wire Wire Line
+	5300 5150 6050 5150
+Wire Wire Line
+	6050 5150 6050 5100
+Connection ~ 5300 4950
+Wire Wire Line
+	5300 4950 5050 4950
 $EndSCHEMATC
